Commit message: change

File: hab_stretch/urdf/stretch_manip_mode.urdf (robot description, URDF)
Before this commit: robot stretch_description, 47 links, 46 joints
Links:
- removed link camera_accel_frame
- removed link camera_accel_optical_frame
- removed link camera_gyro_frame
- removed link camera_gyro_optical_frame
- removed link caster_link
- link base_link: mass 1.1912 -> 1.07237826598; geometry collision mesh filename=package://stretch_description/meshes/base_link.STL; visual mesh filename=package://stretch_description/meshes/base_link.STL
- link camera_link: geometry collision box size=0.02505 0.09 0.025; visual mesh filename=package://realsense2_description/meshes/d435.dae
- link laser: mass 0.0749979022894495 -> 0.0749979022894; geometry collision mesh filename=package://stretch_description/meshes/laser.STL; visual mesh filename=package://stretch_description/meshes/laser.STL
- link link_arm_l0: mass 0.085003260946398 -> 0.101241250325; geometry collision mesh filename=package://stretch_description/meshes/link_arm_l0.STL; visual mesh filename=package://stretch_description/meshes/link_arm_l0.STL
- link link_arm_l1: mass 0.051382 -> 0.0511763619538; geometry collision mesh filename=package://stretch_description/meshes/link_arm_l1.STL; visual mesh filename=package://stretch_description/meshes/link_arm_l1.STL
- link link_arm_l2: mass 0.0571386353275368 -> 0.0569074368576; geometry collision mesh filename=package://stretch_description/meshes/link_arm_l2.STL; visual mesh filename=package://stretch_description/meshes/link_arm_l2.STL
- link link_arm_l3: mass 0.0628927381893134 -> 0.0626921047058; geometry collision mesh filename=package://stretch_description/meshes/link_arm_l3.STL; visual mesh filename=package://stretch_description/meshes/link_arm_l3.STL
- link link_arm_l4: mass 0.068095 -> 0.067652545579; geometry collision mesh filename=package://stretch_description/meshes/link_arm_l4.STL; visual mesh filename=package://stretch_description/meshes/link_arm_l4.STL
- link link_aruco_inner_wrist: mass 0.0 -> 0.000225; geometry collision mesh filename=package://stretch_description/meshes/link_aruco_inner_wrist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; visual mesh filename=package://stretch_description/meshes/link_aruco_inner_wrist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
- link link_aruco_left_base: mass 3.59999999990368e-06 -> 3.5999999999e-06; geometry collision mesh filename=package://stretch_description/meshes/link_aruco_left_base.S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; visual mesh filename=package://stretch_description/meshes/link_aruco_left_base.S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
- link link_aruco_right_base: mass 3.59999999990368e-06 -> 3.5999999999e-06; geometry collision mesh filename=package://stretch_description/meshes/link_aruco_right_base.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; visual mesh filename=package://stretch_description/meshes/link_aruco_right_base.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
- link link_aruco_shoulder: mass 0.0 -> 0.000399141592654; geometry collision mesh filename=package://stretch_description/meshes/link_aruco_shoulder.STL; visual mesh filename=package://stretch_description/meshes/link_aruco_shoulder.STL
- link link_aruco_top_wrist: mass 0.0 -> 0.000225; geometry collision mesh filename=package://stretch_description/meshes/link_aruco_top_wrist.S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; visual mesh filename=package://stretch_description/meshes/link_aruco_top_wrist.S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
- link link_gripper_finger_left: mass 0.0476207785199479 -> 0.0476207785199; geometry collision mesh filename=package://stretch_description/meshes/link_gripper_finger_le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; visual mesh filename=package://stretch_description/meshes/link_gripper_finger_le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
- link link_gripper_finger_right: geometry collision mesh filename=package://stretch_description/meshes/link_gripper_finger_ri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; visual mesh filename=package://stretch_description/meshes/link_gripper_finger_ri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
- link link_gripper_fingertip_left: mass 0.00382160686584851 -> 0.00382160686585; geometry collision mesh filename=package://stretch_description/meshes/link_gripper_fingertip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; visual mesh filename=package://stretch_description/meshes/link_gripper_fingertip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
- link link_gripper_fingertip_right: mass 0.00382160881468841 -> 0.00382160881469; geometry collision mesh filename=package://stretch_description/meshes/link_gripper_fingertip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; visual mesh filename=package://stretch_description/meshes/link_gripper_fingertip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
- link link_head: mass 0.133027236718691 -> 0.129454717596; geometry collision mesh filename=package://stretch_description/meshes/link_head.STL; visual mesh filename=package://stretch_description/meshes/link_head.STL
- link link_head_pan: mass 0.0273764496535409 -> 0.0358583411826; geometry collision mesh filename=package://stretch_description/meshes/link_head_pan.STL; visual mesh filename=package://stretch_description/meshes/link_head_pan.STL
- link link_head_tilt: mass 0.090217113313934 -> 0.0701242408063; geometry collision mesh filename=package://stretch_description/meshes/link_head_tilt.STL; visual mesh filename=package://stretch_description/meshes/link_head_tilt.STL
- link link_left_wheel: mass 0.0042721 -> 0.00356714564938; geometry collision mesh filename=package://stretch_description/meshes/link_left_wheel.STL; visual mesh filename=package://stretch_description/meshes/link_left_wheel.STL
- link link_lift: mass 0.27218 -> 0.444820831236; geometry collision mesh filename=package://stretch_description/meshes/link_lift.STL; visual mesh filename=package://stretch_description/meshes/link_lift.STL
- link link_mast: mass 1.8285 -> 0.749143203376; geometry collision mesh filename=package://stretch_description/meshes/link_mast.STL; visual mesh filename=package://stretch_description/meshes/link_mast.STL
- link link_right_wheel: mass 0.0042721 -> 0.00356714564938; geometry collision mesh filename=package://stretch_description/meshes/link_right_wheel.STL; visual mesh filename=package://stretch_description/meshes/link_right_wheel.STL
- link link_straight_gripper: mass 0.0496384234458284 -> 0.0496384234458; geometry collision mesh filename=package://stretch_description/meshes/link_straight_gripper.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; visual mesh filename=package://stretch_description/meshes/link_straight_gripper.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
- link link_wrist_pitch: mass 0.0701267146295583 -> 0.0701267146296; geometry collision mesh filename=package://stretch_description/meshes/link_wrist_pitch.STL; visual mesh filename=package://stretch_description/meshes/link_wrist_pitch.STL
- link link_wrist_roll: mass 0.00585666394358811 -> 0.00585666394359; geometry collision mesh filename=package://stretch_description/meshes/link_wrist_roll.STL; visual mesh filename=package://stretch_description/meshes/link_wrist_roll.STL
- link link_wrist_yaw: mass 0.0404746907425003 -> 0.0405398981326; geometry collision mesh filename=package://stretch_description/meshes/link_wrist_yaw.STL; visual mesh filename=package://stretch_description/meshes/link_wrist_yaw.STL
- link link_wrist_yaw_bottom: mass 0.0988906816399982 -> 0.09889068164; geometry collision mesh filename=package://stretch_description/meshes/link_wrist_yaw_bottom.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; visual mesh filename=package://stretch_description/meshes/link_wrist_yaw_bottom.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
- link respeaker_base: mass 0.015643 -> 0.00969129410417; geometry collision mesh filename=package://stretch_description/meshes/link_respeaker.STL; visual mesh filename=package://stretch_description/meshes/link_respeaker.STL
Joints:
- removed joint camera_accel_joint
- removed joint camera_accel_optical_joint
- removed joint camera_gyro_joint
- removed joint camera_gyro_optical_joint
- removed joint caster_joint
- joint camera_color_optical_joint: origin xyz=0.0 0.0 0.0 rpy=-1.5707963267948966 0.0 -1.5707963267948966 -> xyz=0.0 0.0 0.0 rpy=-1.57079632679 0.0 -1.57079632679
- joint camera_depth_optical_joint: origin xyz=0.0 0.0 0.0 rpy=-1.5707963267948966 0.0 -1.5707963267948966 -> xyz=0.0 0.0 0.0 rpy=-1.57079632679 0.0 -1.57079632679
- joint camera_infra1_optical_joint: origin xyz=0.0 0.0 0.0 rpy=-1.5707963267948966 0.0 -1.5707963267948966 -> xyz=0.0 0.0 0.0 rpy=-1.57079632679 0.0 -1.57079632679
- joint camera_infra2_optical_joint: origin xyz=0.0 0.0 0.0 rpy=-1.5707963267948966 0.0 -1.5707963267948966 -> xyz=0.0 0.0 0.0 rpy=-1.57079632679 0.0 -1.57079632679
- joint camera_joint: origin xyz=0.02802960503838624 -0.007608222297947431 0.018218494141479257 rpy=0.010658876360659654 -0.0022761048951753793 0.018675317090921212 -> xyz=0.02639642688572102 -0.0089025562918731 0.01841176226710054 rpy=0.0015712819241228975 -0.010836070438404288 -0.04254425710874217
- joint camera_link_joint: origin xyz=0.010600000000000002 0.0175 0.0125 rpy=0.0 0.0 0.0 -> xyz=0.0106 0.0175 0.0125 rpy=0.0 0.0 0.0
- joint joint_arm_l0: origin xyz=0.0 0.0 -0.0137499999991968 rpy=7.63746778746202e-30 -3.80121128864402e-15 2.62707547767438e-15 -> xyz=0.0 0.0 -0.01375 rpy=-3.05317390622e-16 -4.23236224077e-16 -2.68425135229e-17
- joint joint_arm_l1: origin xyz=0.0 0.0 0.0129999999999981 rpy=-7.63746778746202e-30 -7.88860905221012e-31 1.11022302462516e-16 -> xyz=0.0 0.0 0.013 rpy=7.41596560408e-17 1.33876788297e-16 -2.44545873596e-16
- joint joint_arm_l2: origin xyz=0.0 0.0 0.013 rpy=0.0 1.57655765344625e-30 -1.66533453693773e-16 -> xyz=0.0 0.0 0.013 rpy=2.91385731014e-16 4.44300759505e-17 3.25691080516e-16
- joint joint_arm_l3: origin xyz=0.0 0.0 0.013 rpy=7.68831233799385e-30 2.36716479416092e-30 2.29652732251143e-17 -> xyz=0.0 0.0 0.013 rpy=3.5742e-16 3.2123e-16 -2.4565e-16
- joint joint_arm_l4: origin xyz=-0.25956015433181046 -0.0059261537843136765 -0.005557384627505743 rpy=1.5619286973774569 -0.006924580188019336 -1.575847166561953 -> xyz=-0.25446128458494605 0.00025298623412431235 -0.0031376994546148222 rpy=1.5837785805657099 -0.02491831129420552 -1.5856030775202077
- joint joint_aruco_inner_wrist: origin xyz=0.0472499999999947 -0.0119000000000034 -0.0272499999991938 rpy=3.14159265358979 4.23377442363088e-14 3.14159265358979 -> xyz=0.04725 -0.0119 -0.0272499999992 rpy=3.14159265359 4.23377442363e-14 3.14159265359
- joint joint_aruco_left_base: origin xyz=-0.00500000000000014 0.1304972 0.1597482 rpy=0.0 0.0 -1.5707963267949 -> xyz=-0.005 0.1304972 0.1597482 rpy=0.0 0.0 -1.57079632679
- joint joint_aruco_right_base: origin xyz=-0.0015028 -0.1304972 0.1597482 rpy=0.0 0.0 -1.5707963267949 -> xyz=-0.005 -0.1304972 0.1597482 rpy=0.0 0.0 -1.57079632679
- joint joint_aruco_shoulder: origin xyz=-0.0133768876375287 0.0558540528812078 0.0861368272417975 rpy=-1.53998860117704e-29 3.55962409571165e-15 0.0 -> xyz=-0.0133768876375 0.0558540528812 0.0861368272418 rpy=-1.53998860118e-29 3.55962409571e-15 0.0
- joint joint_aruco_top_wrist: origin xyz=0.0472500000000019 0.0292850000000015 0.0 rpy=1.5707963267949 -8.03728587323464e-15 3.14159265358979 -> xyz=0.04725 0.029285 0.0 rpy=1.57079632679 -8.03728587323e-15 3.14159265359
- joint joint_gripper_fingertip_left: origin xyz=0.190596948563868 -0.015 0.0 rpy=1.57079632679496 4.51275387511463e-14 2.60113659715756 -> xyz=0.190596948564 -0.015 0.0 rpy=1.57079632679 4.51275387511e-14 2.60113659716
- joint joint_gripper_fingertip_right: origin xyz=-0.190596948563868 -0.015 0.0 rpy=-1.57079632679483 -3.43320051448326e-14 0.540456056432235 -> xyz=-0.190596948564 -0.015 0.0 rpy=-1.57079632679 -3.43320051448e-14 0.540456056432
- joint joint_head: origin xyz=0.0 1.33 0.0 rpy=1.5707963267949 -1.5707963267949 3.1416 -> xyz=0.0 1.33 0.0 rpy=1.5708 -1.5615 3.1416
- joint joint_head_pan: origin xyz=0.1284513021260868 0.07637128403435504 0.00023722543808071166 rpy=-0.013467967166369273 0.005690738105448956 1.6024957766579377 -> xyz=0.13714093786332454 0.07539709958569715 -0.008416729835197643 rpy=0.006708533220679182 0.010327550569354527 1.5683374379096817
- joint joint_head_tilt: origin xyz=0.0032337815907659225 0.030910701770693223 -0.04783143162927699 rpy=1.5763332066189244 -0.029319157204454882 -0.005080558641851002 -> xyz=-0.00044929845371643323 0.023989180037479706 -0.0546389868277332 rpy=1.5870339278739374 -0.0017951085089351615 0.015184699535185467
- joint joint_laser: origin xyz=0.004 0.0 0.1664 rpy=0.0 0.0 3.1416 -> xyz=0.000502800000001 0.0 0.1664 rpy=0.0 0.0 -3.14159265359
- joint joint_left_wheel: origin xyz=0.0 0.17035 0.0508 rpy=-1.5708 2.6317e-16 -8.2057e-19 -> xyz=-0.00300000000002 0.15765 0.0508 rpy=-1.57079632679 3.16227047921e-31 7.88745438254e-16
- joint joint_lift: origin xyz=-0.037385 0.1666 0.0 rpy=-1.5708 1.5708 0.0 -> xyz=-0.0369217062323 0.1654712 -0.000341653286794 rpy=-1.5707963268 1.56154313753 -6.29420043665e-13
- joint joint_mast: origin xyz=-0.07174416574437388 0.13780491000396983 0.03663931715774088 rpy=1.5780076046568878 0.016499709009588637 -0.007971437955302632 -> xyz=-0.06759654153540276 0.13654203294081094 0.027435318566241755 rpy=1.5675402857854555 -0.027386151150363247 0.015861788024035903
- joint joint_respeaker: origin xyz=0.0 1.37236408874452 0.00303065898329655 rpy=-1.5707963267949 -0.698131700797725 4.93295812652799e-16 -> xyz=1.09074743138e-05 1.36992 0.00303572796911 rpy=1.5707963268 0.0 3.14159265359
- joint joint_right_wheel: origin xyz=0.0 -0.17035 0.0508 rpy=-1.5708 1.2717e-16 4.8006e-17 -> xyz=-0.003 -0.15765 0.0508 rpy=-1.57079632679 -1.11022302463e-16 7.2858385991e-17
- joint joint_straight_gripper: origin xyz=0.0 0.0 0.0155 rpy=3.54987407349455e-30 3.24021254484265e-20 -3.14159265358979 -> xyz=0.0 0.0 0.0155 rpy=3.54987407349e-30 3.24021254484e-20 -3.14159265359
- joint joint_wrist_pitch: origin xyz=0.0 -0.0195500000000002 -0.0247499999999984 rpy=1.5707963267949 -8.12895570882604e-15 -3.14159265358979 -> xyz=0.0 -0.01955 -0.02475 rpy=1.57079632679 -8.12895570883e-15 -3.14159265359
- joint joint_wrist_roll: origin xyz=-0.0188587444076125 -0.0239999999998942 0.01955 rpy=3.14159265358979 1.5707963267949 0.0 -> xyz=-0.0188587444076 -0.0239999999999 0.01955 rpy=3.14159265359 1.57079632679 0.0
- joint joint_wrist_yaw: origin xyz=0.0830000000000654 -0.0307500000000129 0.0 rpy=1.5708 4.2595e-14 2.6415e-15 -> xyz=0.083 -0.03075 0.0 rpy=1.5708 4.2595e-14 2.6415e-15
- joint joint_wrist_yaw_bottom: origin xyz=0.0 0.0 0.0 rpy=-3.14159265358979 1.13367999021379e-14 1.57079632679489 -> xyz=0.0 0.0 0.0 rpy=-3.14159265359 1.13367999021e-14 1.57079632679
