Commit message: All Urdfs

File: robot/urdf/stretch5.urdf (robot description, URDF)
Before this commit: robot stretch_description, 42 links, 41 joints
Links:
- removed link link_gripper
- added link fake_link_x, mass 0.749143203376
- added link link_straight_gripper, mass 0.147853; collision mesh filename=package://stretch_description/meshes/link_straight_gripper.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; visual mesh filename=package://stretch_description/meshes/link_straight_gripper.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
- added link link_wrist_pitch, mass 0.208129; collision mesh filename=package://stretch_description/meshes/link_wrist_pitch.STL; visual mesh filename=package://stretch_description/meshes/link_wrist_pitch.STL
- added link link_wrist_roll, mass 0.01528; collision mesh filename=package://stretch_description/meshes/link_wrist_roll.STL; visual mesh filename=package://stretch_description/meshes/link_wrist_roll.STL
- added link link_wrist_yaw_bottom, mass 0.24284; collision mesh filename=package://stretch_description/meshes/link_wrist_yaw_bottom.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; visual mesh filename=package://stretch_description/meshes/link_wrist_yaw_bottom.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
- link base_link: mass 1.0723782659782 -> 17.384389
- link laser: mass 0.0749979022894495 -> 0.216007
- link link_arm_l0: mass 0.101241250325294 -> 0.427734
- link link_arm_l1: mass 0.0511763619538321 -> 0.113658
- link link_arm_l2: mass 0.0569074368576238 -> 0.130565
- link link_arm_l3: mass 0.0626921047058405 -> 0.146817
- link link_arm_l4: mass 0.0676525455789735 -> 0.235626
- link link_gripper_finger_left: mass 0.0476207785199474 -> 0.06; geometry collision mesh filename=package://stretch_description/meshes/link_gripper_finger_le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; visual mesh filename=package://stretch_description/meshes/link_gripper_finger_le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
- link link_gripper_finger_right: mass 0.0476207785199481 -> 0.06; geometry collision mesh filename=package://stretch_description/meshes/link_gripper_finger_ri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; visual mesh filename=package://stretch_description/meshes/link_gripper_finger_ri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
- link link_gripper_fingertip_left: mass 0.00382159917455729 -> 0.003822
- link link_gripper_fingertip_right: mass 0.00382160037319545 -> 0.003822
- link link_head: mass 0.129454717596498 -> 0.681871
- link link_head_pan: mass 0.035858341182617 -> 0.062462
- link link_head_tilt: mass 0.0701242408063442 -> 0.283548
- link link_left_wheel: mass 0.01 -> 0.20773
- link link_lift: mass 0.444820831236007 -> 1.987167
- link link_mast: mass 0.749143203376401 -> 1.764017
- link link_right_wheel: mass 0.01 -> 0.20773
- link link_wrist_yaw: mass 0.0405398981326229 -> 0.054422
- link respeaker_base: mass 0.00969129410417277 -> 0.025175; geometry collision mesh filename=package://stretch_description/meshes/respeaker_base.STL; visual mesh filename=package://stretch_description/meshes/respeaker_base.STL
Joints:
- removed joint joint_gripper
- added joint joint_fake: type prismatic, parent base_link, child fake_link_x, origin xyz=0. 0. 0. rpy=0. 0. 0., axis 1.0 0.0 0.0, limit lower=-1.0 upper=1.1 effort=100.0 velocity=1.0
- added joint joint_straight_gripper: type fixed, parent link_wrist_roll, child link_straight_gripper, origin xyz=0.0 0.0 0.0155 rpy=3.54987407349455e-30 3.24021254484265e-20 -3.14159265358979, axis 0.0 0.0 0.0
- added joint joint_wrist_pitch: type revolute, parent link_wrist_yaw_bottom, child link_wrist_pitch, origin xyz=0.0 -0.0195500000000002 -0.0247499999999984 rpy=1.5707963267949 -8.12895570882604e-15 -3.14159265358979, axis 0.0 0.0 -1.0, limit lower=-1.57 upper=0.56 effort=100.0 velocity=1.0
- added joint joint_wrist_roll: type revolute, parent link_wrist_pitch, child link_wrist_roll, origin xyz=-0.0188587444076125 -0.0239999999998942 0.01955 rpy=3.14159265358979 1.5707963267949 0.0, axis 0.0 0.0 1.0, limit lower=-3.14 upper=3.14 effort=100.0 velocity=1.0
- added joint joint_wrist_yaw_bottom: type fixed, parent link_wrist_yaw, child link_wrist_yaw_bottom, origin xyz=0.0 0.0 0.0 rpy=-3.14159265358979 1.13367999021379e-14 1.57079632679489, axis 0.0 0.0 0.0
- joint camera_joint: origin xyz=0.027473873466743973 -0.007933957203986762 0.01836984283354483 rpy=0.0016751704736353863 -0.011615736976204882 0.007014423573473042 -> xyz=0.028188772272801907 -0.007564712173205754 0.017944882096133475 rpy=0.004350212950992322 0.0034525753069547527 0.017907303224988517
- joint joint_arm_l0: origin xyz=0.0 0.0 -0.0137499999999938 rpy=-3.05317390622457e-16 -4.23236224076729e-16 -2.68425135229209e-17 -> xyz=0.0 0.0 -0.0137499999991968 rpy=7.63746778746202e-30 -3.80121128864402e-15 2.62707547767438e-15
- joint joint_arm_l1: origin xyz=0.0 0.0 0.013 rpy=7.41596560408007e-17 1.33876788296791e-16 -2.44545873596083e-16 -> xyz=0.0 0.0 0.0129999999999981 rpy=-7.63746778746202e-30 -7.88860905221012e-31 1.11022302462516e-16
- joint joint_arm_l2: origin xyz=0.0 0.0 0.013 rpy=2.91385731014123e-16 4.44300759504684e-17 3.25691080516352e-16 -> xyz=0.0 0.0 0.013 rpy=0.0 1.57655765344625e-30 -1.66533453693773e-16
- joint joint_arm_l3: origin xyz=0.0 0.0 0.013 rpy=3.5742e-16 3.2123e-16 -2.4565e-16 -> xyz=0.0 0.0 0.013 rpy=7.68831233799385e-30 2.36716479416092e-30 2.29652732251143e-17
- joint joint_arm_l4: origin xyz=-0.25196873816616694 0.0013913799655517999 -0.00662345856085944 rpy=1.5907891510357897 -0.03915147163900001 -1.6208501453312254 -> xyz=-0.2523079099923315 -0.00046358158197051135 -0.006180072447490051 rpy=1.5851841389128425 -0.008966074572395621 -1.5866239497902528
- joint joint_aruco_right_base: origin xyz=-0.00500000000000014 -0.1304972 0.1597482 rpy=0.0 0.0 -1.5707963267949 -> xyz=-0.0015028 -0.1304972 0.1597482 rpy=0.0 0.0 -1.5707963267949
- joint joint_grasp_center: origin xyz=-0.205478 0.0 -0.138154 rpy=0.0 0.0 3.141579 -> xyz=0.0 0.0 0.23 rpy=-1.5707963267949 -1.5707963267949 0.0; parent link_gripper -> link_straight_gripper
- joint joint_gripper_finger_left: axis 0.0 0.0 1.0 -> 0.0 0.0 -1.0; origin xyz=-0.047231 -0.010151 -0.04679 rpy=2.1762e-15 0.5236 3.1416 -> xyz=0.018599 0.003 0.033689 rpy=1.5708 -1.5708 0.0; parent link_gripper -> link_straight_gripper
- joint joint_gripper_finger_right: origin xyz=-0.047231 0.010049 -0.04679 rpy=3.1416 -0.5236 1.2943e-15 -> xyz=-0.018599 0.003 0.033689 rpy=1.5708 1.5708 0.0; parent link_gripper -> link_straight_gripper
- joint joint_gripper_fingertip_left: origin xyz=0.171099 0.014912 0.0 rpy=-1.5708 -4.774e-15 -2.5545 -> xyz=0.190596948563868 -0.015 0.0 rpy=1.57079632679496 4.51275387511463e-14 2.60113659715756
- joint joint_gripper_fingertip_right: origin xyz=-0.171099 -0.014912 0.0 rpy=-1.5708 -2.0539e-15 0.58705 -> xyz=-0.190596948563868 -0.015 0.0 rpy=-1.57079632679483 -3.43320051448326e-14 0.540456056432235
- joint joint_head: origin xyz=0.0 1.33 0.0 rpy=1.5708 -1.5615 3.1416 -> xyz=0.0 1.33 0.0 rpy=1.5707963267949 -1.5707963267949 3.1416
- joint joint_head_pan: origin xyz=0.13895476234644444 0.07638226882137976 -0.007346107154901064 rpy=0.015514956127904081 0.018602518596500417 1.6351927362304166 -> xyz=0.13325570978545617 0.07617617446959961 -0.009351286218560623 rpy=0.01100262211911233 0.016732815421323766 1.573854796890386
- joint joint_head_tilt: origin xyz=-0.003735897943321004 0.023195008877475276 -0.052980398024184326 rpy=1.5623704297642063 0.028915120156655316 0.01511995981348627 -> xyz=-0.006034037729667192 0.024051664840607265 -0.05437206063104133 rpy=1.5467189102976846 0.03568929327401138 0.06774098088428002
- joint joint_laser: origin xyz=0.000502800000000914 0.0 0.1664 rpy=0.0 0.0 -3.14159265358979 -> xyz=0.004 0.0 0.1664 rpy=0.0 0.0 3.1416
- joint joint_left_wheel: origin xyz=-0.003 0.15765 0.05 rpy=-1.5707963267949 3.16227047920818e-31 7.88745438253713e-16 -> xyz=0.0 0.17035 0.0508 rpy=-1.5708 2.6317e-16 -8.2057e-19
- joint joint_lift: limit lower=-0.1033 upper=0.9967 effort=100.0 velocity=1.0 -> lower=0.0 upper=1.1 effort=100.0 velocity=1.0; origin xyz=-0.0369217062323472 0.268771199999996 -0.000341653286793524 rpy=-1.57079632679552 1.5615431375292 -6.2942004366467e-13 -> xyz=-0.037385 0.1666 0.0 rpy=-1.5708 1.5708 0.0
- joint joint_mast: origin xyz=-0.07444652084656547 0.1370485367923482 0.026461832859242185 rpy=1.5746294433173749 0.01253227831941528 0.05018860915999327 -> xyz=-0.06886239813360509 0.13725755297906447 0.025143215009302215 rpy=1.5725304449603004 0.0027932103811125764 0.013336895699597295; parent base_link -> fake_link_x
- joint joint_respeaker: origin xyz=1.09074743137871e-05 1.36992 0.00303572796911382 rpy=1.57079632679553 0.0 3.14159265358916 -> xyz=0.0 1.37236408874452 0.00303065898329655 rpy=-1.5707963267949 -0.698131700797725 4.93295812652799e-16
- joint joint_right_wheel: origin xyz=-0.003 -0.15765 0.05 rpy=-1.57079632679489 -1.11022302462516e-16 7.28583859910277e-17 -> xyz=0.0 -0.17035 0.0508 rpy=-1.5708 1.2717e-16 4.8006e-17
- joint joint_wrist_yaw: origin xyz=0.083 -0.03075 0.0 rpy=1.5708 4.2595e-14 2.6415e-15 -> xyz=0.0830000000000654 -0.0307500000000129 0.0 rpy=1.5708 4.2595e-14 2.6415e-15
