Commit message: Changed few more filenames

File: robot/urdf/stretch.urdf (robot description, URDF)
Before this commit: robot stretch_description, 40 links, 39 joints
Links:
- added link camera_accel_frame
- added link camera_accel_optical_frame
- added link camera_gyro_frame
- added link camera_gyro_optical_frame
- added link caster_link, mass 0.01; collision sphere radius=0.032; visual mesh filename=package://stretch_description/meshes/omni_wheel_m.STL
- added link link_grasp_center
- link base_link: mass 1.07237826598 -> 17.384389
- link laser: mass 0.0749979022894 -> 0.216007
- link link_arm_l0: mass 0.101241250325 -> 0.427734
- link link_arm_l1: mass 0.0511763619538 -> 0.113658
- link link_arm_l2: mass 0.0569074368576 -> 0.130565
- link link_arm_l3: mass 0.0626921047058 -> 0.146817
- link link_arm_l4: mass 0.067652545579 -> 0.235626
- link link_aruco_inner_wrist: mass 0.000225 -> 0.0
- link link_aruco_left_base: mass 3.5999999999e-06 -> 3.59999999990368e-06
- link link_aruco_right_base: mass 3.5999999999e-06 -> 3.59999999990368e-06
- link link_aruco_shoulder: mass 0.000399141592654 -> 0.0
- link link_aruco_top_wrist: mass 0.000225 -> 0.0
- link link_gripper_finger_left: mass 0.0476207785199 -> 0.06
- link link_gripper_finger_right: mass 0.047621 -> 0.06
- link link_gripper_fingertip_left: mass 0.00382160686585 -> 0.003822
- link link_gripper_fingertip_right: mass 0.00382160881469 -> 0.003822
- link link_head: mass 0.129454717596 -> 0.681871
- link link_head_pan: mass 0.0358583411826 -> 0.062462
- link link_head_tilt: mass 0.0701242408063 -> 0.283548
- link link_left_wheel: mass 0.00356714564938 -> 0.20773
- link link_lift: mass 0.444820831236 -> 1.987167
- link link_mast: mass 0.749143203376 -> 1.764017
- link link_right_wheel: mass 0.00356714564938 -> 0.20773
- link link_straight_gripper: mass 0.0496384234458 -> 0.147853
- link link_wrist_pitch: mass 0.0701267146296 -> 0.208129
- link link_wrist_roll: mass 0.00585666394359 -> 0.01528
- link link_wrist_yaw: mass 0.0405398981326 -> 0.054422
- link link_wrist_yaw_bottom: mass 0.09889068164 -> 0.24284
- link respeaker_base: mass 0.00969129410417 -> 0.025175; geometry collision mesh filename=package://stretch_description/meshes/respeaker_base.STL; visual mesh filename=package://stretch_description/meshes/respeaker_base.STL
Joints:
- added joint camera_accel_joint: type fixed, parent camera_link, child camera_accel_frame, origin xyz=-0.01174 -0.00552 0.0051 rpy=0.0 0.0 0.0
- added joint camera_accel_optical_joint: type fixed, parent camera_accel_frame, child camera_accel_optical_frame, origin xyz=0.0 0.0 0.0 rpy=-1.5707963267948966 0.0 -1.5707963267948966
- added joint camera_gyro_joint: type fixed, parent camera_link, child camera_gyro_frame, origin xyz=-0.01174 -0.00552 0.0051 rpy=0.0 0.0 0.0
- added joint camera_gyro_optical_joint: type fixed, parent camera_gyro_frame, child camera_gyro_optical_frame, origin xyz=0.0 0.0 0.0 rpy=-1.5707963267948966 0.0 -1.5707963267948966
- added joint caster_joint: type fixed, parent base_link, child caster_link, origin xyz=-0.245 0.0 0.032 rpy=-1.5707963267948966 0.0 0.0, axis 0.0 0.0 1.0
- added joint joint_grasp_center: type fixed, parent link_straight_gripper, child link_grasp_center, origin xyz=0.0 0.0 0.23 rpy=-1.5707963267949 -1.5707963267949 0.0
- joint camera_color_optical_joint: origin xyz=0.0 0.0 0.0 rpy=-1.57079632679 0.0 -1.57079632679 -> xyz=0.0 0.0 0.0 rpy=-1.5707963267948966 0.0 -1.5707963267948966
- joint camera_depth_optical_joint: origin xyz=0.0 0.0 0.0 rpy=-1.57079632679 0.0 -1.57079632679 -> xyz=0.0 0.0 0.0 rpy=-1.5707963267948966 0.0 -1.5707963267948966
- joint camera_infra1_optical_joint: origin xyz=0.0 0.0 0.0 rpy=-1.57079632679 0.0 -1.57079632679 -> xyz=0.0 0.0 0.0 rpy=-1.5707963267948966 0.0 -1.5707963267948966
- joint camera_infra2_optical_joint: origin xyz=0.0 0.0 0.0 rpy=-1.57079632679 0.0 -1.57079632679 -> xyz=0.0 0.0 0.0 rpy=-1.5707963267948966 0.0 -1.5707963267948966
- joint camera_joint: origin xyz=0.02639642688572102 -0.0089025562918731 0.01841176226710054 rpy=0.0015712819241228975 -0.010836070438404288 -0.04254425710874217 -> xyz=0.028188772272801907 -0.007564712173205754 0.017944882096133475 rpy=0.004350212950992322 0.0034525753069547527 0.017907303224988517
- joint camera_link_joint: origin xyz=0.0106 0.0175 0.0125 rpy=0.0 0.0 0.0 -> xyz=0.010600000000000002 0.0175 0.0125 rpy=0.0 0.0 0.0
- joint joint_arm_l0: origin xyz=0.0 0.0 -0.01375 rpy=-3.05317390622e-16 -4.23236224077e-16 -2.68425135229e-17 -> xyz=0.0 0.0 -0.0137499999991968 rpy=7.63746778746202e-30 -3.80121128864402e-15 2.62707547767438e-15
- joint joint_arm_l1: origin xyz=0.0 0.0 0.013 rpy=7.41596560408e-17 1.33876788297e-16 -2.44545873596e-16 -> xyz=0.0 0.0 0.0129999999999981 rpy=-7.63746778746202e-30 -7.88860905221012e-31 1.11022302462516e-16
- joint joint_arm_l2: origin xyz=0.0 0.0 0.013 rpy=2.91385731014e-16 4.44300759505e-17 3.25691080516e-16 -> xyz=0.0 0.0 0.013 rpy=0.0 1.57655765344625e-30 -1.66533453693773e-16
- joint joint_arm_l3: origin xyz=0.0 0.0 0.013 rpy=3.5742e-16 3.2123e-16 -2.4565e-16 -> xyz=0.0 0.0 0.013 rpy=7.68831233799385e-30 2.36716479416092e-30 2.29652732251143e-17
- joint joint_arm_l4: origin xyz=-0.25446128458494605 0.00025298623412431235 -0.0031376994546148222 rpy=1.5837785805657099 -0.02491831129420552 -1.5856030775202077 -> xyz=-0.2523079099923315 -0.00046358158197051135 -0.006180072447490051 rpy=1.5851841389128425 -0.008966074572395621 -1.5866239497902528
- joint joint_aruco_inner_wrist: origin xyz=0.04725 -0.0119 -0.0272499999992 rpy=3.14159265359 4.23377442363e-14 3.14159265359 -> xyz=0.0472499999999947 -0.0119000000000034 -0.0272499999991938 rpy=3.14159265358979 4.23377442363088e-14 3.14159265358979
- joint joint_aruco_left_base: origin xyz=-0.005 0.1304972 0.1597482 rpy=0.0 0.0 -1.57079632679 -> xyz=-0.00500000000000014 0.1304972 0.1597482 rpy=0.0 0.0 -1.5707963267949
- joint joint_aruco_right_base: origin xyz=-0.005 -0.1304972 0.1597482 rpy=0.0 0.0 -1.57079632679 -> xyz=-0.0015028 -0.1304972 0.1597482 rpy=0.0 0.0 -1.5707963267949
- joint joint_aruco_shoulder: origin xyz=-0.0133768876375 0.0558540528812 0.0861368272418 rpy=-1.53998860118e-29 3.55962409571e-15 0.0 -> xyz=-0.0133768876375287 0.0558540528812078 0.0861368272417975 rpy=-1.53998860117704e-29 3.55962409571165e-15 0.0
- joint joint_aruco_top_wrist: origin xyz=0.04725 0.029285 0.0 rpy=1.57079632679 -8.03728587323e-15 3.14159265359 -> xyz=0.0472500000000019 0.0292850000000015 0.0 rpy=1.5707963267949 -8.03728587323464e-15 3.14159265358979
- joint joint_gripper_fingertip_left: origin xyz=0.190596948564 -0.015 0.0 rpy=1.57079632679 4.51275387511e-14 2.60113659716 -> xyz=0.190596948563868 -0.015 0.0 rpy=1.57079632679496 4.51275387511463e-14 2.60113659715756
- joint joint_gripper_fingertip_right: origin xyz=-0.190596948564 -0.015 0.0 rpy=-1.57079632679 -3.43320051448e-14 0.540456056432 -> xyz=-0.190596948563868 -0.015 0.0 rpy=-1.57079632679483 -3.43320051448326e-14 0.540456056432235
- joint joint_head: origin xyz=0.0 1.33 0.0 rpy=1.5708 -1.5615 3.1416 -> xyz=0.0 1.33 0.0 rpy=1.5707963267949 -1.5707963267949 3.1416
- joint joint_head_pan: origin xyz=0.13714093786332454 0.07539709958569715 -0.008416729835197643 rpy=0.006708533220679182 0.010327550569354527 1.5683374379096817 -> xyz=0.13325570978545617 0.07617617446959961 -0.009351286218560623 rpy=0.01100262211911233 0.016732815421323766 1.573854796890386
- joint joint_head_tilt: origin xyz=-0.00044929845371643323 0.023989180037479706 -0.0546389868277332 rpy=1.5870339278739374 -0.0017951085089351615 0.015184699535185467 -> xyz=-0.006034037729667192 0.024051664840607265 -0.05437206063104133 rpy=1.5467189102976846 0.03568929327401138 0.06774098088428002
- joint joint_laser: origin xyz=0.000502800000001 0.0 0.1664 rpy=0.0 0.0 -3.14159265359 -> xyz=0.004 0.0 0.1664 rpy=0.0 0.0 3.1416
- joint joint_left_wheel: origin xyz=-0.00300000000002 0.15765 0.0508 rpy=-1.57079632679 3.16227047921e-31 7.88745438254e-16 -> xyz=0.0 0.17035 0.0508 rpy=-1.5708 2.6317e-16 -8.2057e-19
- joint joint_lift: origin xyz=-0.0369217062323 0.1654712 -0.000341653286794 rpy=-1.5707963268 1.56154313753 -6.29420043665e-13 -> xyz=-0.037385 0.1666 0.0 rpy=-1.5708 1.5708 0.0
- joint joint_mast: origin xyz=-0.06759654153540276 0.13654203294081094 0.027435318566241755 rpy=1.5675402857854555 -0.027386151150363247 0.015861788024035903 -> xyz=-0.06886239813360509 0.13725755297906447 0.025143215009302215 rpy=1.5725304449603004 0.0027932103811125764 0.013336895699597295
- joint joint_respeaker: origin xyz=1.09074743138e-05 1.36992 0.00303572796911 rpy=1.5707963268 0.0 3.14159265359 -> xyz=0.0 1.37236408874452 0.00303065898329655 rpy=-1.5707963267949 -0.698131700797725 4.93295812652799e-16
- joint joint_right_wheel: origin xyz=-0.003 -0.15765 0.0508 rpy=-1.57079632679 -1.11022302463e-16 7.2858385991e-17 -> xyz=0.0 -0.17035 0.0508 rpy=-1.5708 1.2717e-16 4.8006e-17
- joint joint_straight_gripper: origin xyz=0.0 0.0 0.0155 rpy=3.54987407349e-30 3.24021254484e-20 -3.14159265359 -> xyz=0.0 0.0 0.0155 rpy=3.54987407349455e-30 3.24021254484265e-20 -3.14159265358979
- joint joint_wrist_pitch: origin xyz=0.0 -0.01955 -0.02475 rpy=1.57079632679 -8.12895570883e-15 -3.14159265359 -> xyz=0.0 -0.0195500000000002 -0.0247499999999984 rpy=1.5707963267949 -8.12895570882604e-15 -3.14159265358979
- joint joint_wrist_roll: origin xyz=-0.0188587444076 -0.0239999999999 0.01955 rpy=3.14159265359 1.57079632679 0.0 -> xyz=-0.0188587444076125 -0.0239999999998942 0.01955 rpy=3.14159265358979 1.5707963267949 0.0
- joint joint_wrist_yaw: origin xyz=0.083 -0.03075 0.0 rpy=1.5708 4.2595e-14 2.6415e-15 -> xyz=0.0830000000000654 -0.0307500000000129 0.0 rpy=1.5708 4.2595e-14 2.6415e-15
- joint joint_wrist_yaw_bottom: origin xyz=0.0 0.0 0.0 rpy=-3.14159265359 1.13367999021e-14 1.57079632679 -> xyz=0.0 0.0 0.0 rpy=-3.14159265358979 1.13367999021379e-14 1.57079632679489

Commit message: making some changes

File: robot/urdf/stretch.urdf (robot description, URDF)
Before this commit: robot stretch_description, 46 links, 45 joints
Joints:
- joint camera_joint: origin xyz=0.028188772272801907 -0.007564712173205754 0.017944882096133475 rpy=0.004350212950992322 0.0034525753069547527 0.017907303224988517 -> xyz=0.02619219623036331 -0.00907998840588666 0.017504180222345376 rpy=0.024000002807284544 -0.008300456177192217 -0.05827310651731734
- joint joint_arm_l4: origin xyz=-0.2523079099923315 -0.00046358158197051135 -0.006180072447490051 rpy=1.5851841389128425 -0.008966074572395621 -1.5866239497902528 -> xyz=-0.25346046622553026 -0.0006888955385321449 -0.009067467536432347 rpy=1.5723623435010765 0.02018571874175068 -1.5695989194351543
- joint joint_head_pan: origin xyz=0.13325570978545617 0.07617617446959961 -0.009351286218560623 rpy=0.01100262211911233 0.016732815421323766 1.573854796890386 -> xyz=0.12653591644065892 0.06996300447388382 -0.007502567186114471 rpy=-0.013482085643258484 0.008351178824350214 1.5828756850605683
- joint joint_head_tilt: origin xyz=-0.006034037729667192 0.024051664840607265 -0.05437206063104133 rpy=1.5467189102976846 0.03568929327401138 0.06774098088428002 -> xyz=-0.010551572466977533 0.03117939300009126 -0.05286298183491632 rpy=1.6180532800825063 -0.03979025166173167 0.0358699222168261
- joint joint_mast: origin xyz=-0.06886239813360509 0.13725755297906447 0.025143215009302215 rpy=1.5725304449603004 0.0027932103811125764 0.013336895699597295 -> xyz=-0.0724940356922689 0.1396132937867568 0.021697509564934978 rpy=1.5742152551827593 0.023130319841277114 0.033874711475578384

Commit message: update docs

File: robot/urdf/stretch.urdf (robot description, URDF)
Before this commit: robot stretch_description, 46 links, 45 joints
Links:
- added link base_imu, mass 0.00092; collision mesh filename=package://stretch_description/meshes/base_imu.STL; visual mesh filename=package://stretch_description/meshes/base_imu.STL
Joints:
- added joint joint_base_imu: type fixed, parent base_link, child base_imu, origin xyz=-0.12838 0.0031592 0.1474 rpy=-3.1416 0.0 -1.5708, axis 0.0 0.0 0.0
- joint camera_joint: origin xyz=0.02619219623036331 -0.00907998840588666 0.017504180222345376 rpy=0.024000002807284544 -0.008300456177192217 -0.05827310651731734 -> xyz=0.02607886806949255 -0.009314618418488976 0.01895352363443432 rpy=0.023237650152550023 -0.007836420162175894 -0.03265182473345039
- joint joint_arm_l4: origin xyz=-0.25346046622553026 -0.0006888955385321449 -0.009067467536432347 rpy=1.5723623435010765 0.02018571874175068 -1.5695989194351543 -> xyz=-0.2551902995196521 -0.004587477527919949 -0.0067835018335551 rpy=1.5947532545223841 0.04310809856221964 -1.5634231107732015
- joint joint_head_pan: origin xyz=0.12653591644065892 0.06996300447388382 -0.007502567186114471 rpy=-0.013482085643258484 0.008351178824350214 1.5828756850605683 -> xyz=0.13453874536738517 0.07312635667870605 -0.011180608315312722 rpy=-0.0030738562300043934 0.0073597460057950315 1.5950287113810948
- joint joint_head_tilt: origin xyz=-0.010551572466977533 0.03117939300009126 -0.05286298183491632 rpy=1.6180532800825063 -0.03979025166173167 0.0358699222168261 -> xyz=-0.004901621230908064 0.03035253842258606 -0.04865203443747947 rpy=1.6195958295464712 0.005886338648440459 0.060555244385694935
- joint joint_mast: origin xyz=-0.0724940356922689 0.1396132937867568 0.021697509564934978 rpy=1.5742152551827593 0.023130319841277114 0.033874711475578384 -> xyz=-0.07198330012654981 0.13523123076717533 0.022499411208387422 rpy=1.5697469575590208 0.0014651016685551799 0.024884147606998232
